File: kicad-host-mvp/generated/external-router-output/desktop-air-monitor-krt-routed.kicad_pcb (KiCad board)
At the start: 2 copper layers, 92 x 64 mm, 5 parts

Commit message: 更新
Routing:
- net 5V: track 116.3 -> 118.2 mm

Commit message: update
Routing:
- net 5V: track 118.2 -> 116.3 mm
